File: PCB_MP/PCB_MP_09/PCB_MP_09.kicad_pcb (KiCad board)
At the start: 2 copper layers, 21 parts, among them J1 inputs, U1 74LS151, U10 74HC595, U11 74LS153, U12 74LS153, U13 74LS153, U14 74LS153, U15 74LS153, U16 74LS153, U17 74HC595, U18 74LS151, U19 74HC595, U2 74LS153, U20 74LS151, U3 74LS153, U4 74LS153, U5 74HC595, U6 74LS153, U7 74LS153, U8 74LS153, U9 74LS151

Commit message: schematics: Bus architecture for config and switch bits is used
Parts:
- added U21: ESP32-WROOM-32E, RF_Module:ESP32-WROOM-32D, F.Cu at (234.2, 109.9)
Connections:
- U1 pad 7: unconnected-(U1-~{E}-Pad7) -> GND
- U10 pad 11: unconnected-(U10-SRCLK-Pad11) -> /SRCLK
- U10 pad 12: unconnected-(U10-RCLK-Pad12) -> /RCLK
- U10 pad 14: unconnected-(U10-SER-Pad14) -> /SER
- U10 pad 8: unconnected-(U10-GND-Pad8) -> GND
- U11 pad 3: /4to1mux/I3a_2 -> O/P_L3
- U11 pad 4: /4to1mux/I2a_2 -> O/P_L1
- U12 pad 3: /4to1mux/I3a_2 -> O/P_L3
- U12 pad 4: /4to1mux/I2a_2 -> O/P_L1
- U13 pad 3: /4to1mux/I3a_2 -> O/P_L3
- U13 pad 4: /4to1mux/I2a_2 -> O/P_L1
- U14 pad 3: /4to1mux/I3a_3 -> O/P_L2
- U14 pad 4: /4to1mux/I2a_3 -> O/P_L1
- U14 pad 5: /4to1mux/I1a_3 -> O/P_L0
- U15 pad 3: /4to1mux/I3a_3 -> O/P_L2
- U15 pad 4: /4to1mux/I2a_3 -> O/P_L1
- U15 pad 5: /4to1mux/I1a_3 -> O/P_L0
- U16 pad 3: /4to1mux/I3a_3 -> O/P_L2
- U16 pad 4: /4to1mux/I2a_3 -> O/P_L1
- U16 pad 5: /4to1mux/I1a_3 -> O/P_L0
- U17 pad 11: unconnected-(U17-SRCLK-Pad11) -> /SRCLK
- U17 pad 12: unconnected-(U17-RCLK-Pad12) -> /RCLK
- U17 pad 14: unconnected-(U17-SER-Pad14) -> /SER
- U19 pad 11: unconnected-(U19-SRCLK-Pad11) -> /SRCLK
- U19 pad 12: unconnected-(U19-RCLK-Pad12) -> /RCLK
- U19 pad 14: unconnected-(U19-SER-Pad14) -> /SER
- U2 pad 3: /4to1mux/I3a_0 -> O/P_L3
- U2 pad 4: /4to1mux/I2a_0 -> O/P_L2
- U2 pad 5: /4to1mux/I1a_0 -> O/P_L1
- U3 pad 3: /4to1mux/I3a_0 -> O/P_L3
- U3 pad 4: /4to1mux/I2a_0 -> O/P_L2
- U3 pad 5: /4to1mux/I1a_0 -> O/P_L1
- U4 pad 3: /4to1mux/I3a_0 -> O/P_L3
- U4 pad 4: /4to1mux/I2a_0 -> O/P_L2
- U4 pad 5: /4to1mux/I1a_0 -> O/P_L1
- U5 pad 11: unconnected-(U5-SRCLK-Pad11) -> /SRCLK
- U5 pad 12: unconnected-(U5-RCLK-Pad12) -> /RCLK
- U5 pad 13: unconnected-(U5-~{OE}-Pad13) -> GND
- U5 pad 14: unconnected-(U5-SER-Pad14) -> /SER
- U6 pad 3: /4to1mux/I3a_1 -> O/P_L3
- U6 pad 4: /4to1mux/I2a_1 -> O/P_L2
- U7 pad 3: /4to1mux/I3a_1 -> O/P_L3
- U7 pad 4: /4to1mux/I2a_1 -> O/P_L2
- U8 pad 3: /4to1mux/I3a_1 -> O/P_L3
- U8 pad 4: /4to1mux/I2a_1 -> O/P_L2
- U9 pad 7: unconnected-(U9-~{E}-Pad7) -> GND

Commit message: Logisim: 8bit sipo registers included:: Schematics:switch matrix regs connected
Parts:
- added U22: 74HC595, Package_DIP:DIP-16_W7.62mm_LongPads, F.Cu at (224.9, 132.3)
- added U23: 74HC595, Package_DIP:DIP-16_W7.62mm_LongPads, F.Cu at (242.1, 133.1)
- added U24: 74HC595, Package_DIP:DIP-16_W7.62mm_LongPads, F.Cu at (253.7, 133.1)
- added U25: 74HC595, Package_DIP:DIP-16_W7.62mm_LongPads, F.Cu at (265.3, 133.1)
Connections:
- U10 pad 13: unconnected-(U10-~{OE}-Pad13) -> /OE_1
- U11 pad 14: unconnected-(U11-S0-Pad14) -> /4to1mux/QE_12
- U11 pad 2: unconnected-(U11-S1-Pad2) -> /4to1mux/QF_13
- U12 pad 14: unconnected-(U12-S0-Pad14) -> /4to1mux/QG_14
- U12 pad 2: unconnected-(U12-S1-Pad2) -> /4to1mux/QH_15
- U13 pad 14: unconnected-(U13-S0-Pad14) -> /4to1mux/QA_16
- U13 pad 2: unconnected-(U13-S1-Pad2) -> /4to1mux/QB_17
- U14 pad 14: unconnected-(U14-S0-Pad14) -> /4to1mux/QC_18
- U14 pad 2: unconnected-(U14-S1-Pad2) -> /4to1mux/QD_19
- U15 pad 14: unconnected-(U15-S0-Pad14) -> /4to1mux/QE_20
- U15 pad 2: unconnected-(U15-S1-Pad2) -> /4to1mux/QF_21
- U16 pad 14: unconnected-(U16-S0-Pad14) -> /4to1mux/QG_22
- U16 pad 2: unconnected-(U16-S1-Pad2) -> /4to1mux/QH_23
- U17 pad 13: unconnected-(U17-~{OE}-Pad13) -> /OE_2
- U19 pad 13: GND -> /OE_3
- U2 pad 14: unconnected-(U2-S0-Pad14) -> /4to1mux/QA_00
- U2 pad 2: unconnected-(U2-S1-Pad2) -> /4to1mux/QB_01
- U21 pad 13: unconnected-(U21-IO14-Pad13) -> /SRCLK
- U21 pad 16: unconnected-(U21-IO13-Pad16) -> /SER
- U21 pad 23: unconnected-(U21-IO15-Pad23) -> /RCLK
- U21 pad 27: unconnected-(U21-IO16-Pad27) -> /OE_0
- U21 pad 28: unconnected-(U21-IO17-Pad28) -> /OE_1
- U21 pad 30: unconnected-(U21-IO18-Pad30) -> /OE_2
- U21 pad 31: unconnected-(U21-IO19-Pad31) -> /OE_3
- U21 pad 33: unconnected-(U21-IO21-Pad33) -> SER_sc
- U3 pad 14: unconnected-(U3-S0-Pad14) -> /4to1mux/QC_02
- U3 pad 2: unconnected-(U3-S1-Pad2) -> /4to1mux/QD_03
- U4 pad 14: unconnected-(U4-S0-Pad14) -> /4to1mux/QE_04
- U4 pad 2: unconnected-(U4-S1-Pad2) -> /4to1mux/QF_05
- U5 pad 13: GND -> /OE_0
- U6 pad 14: unconnected-(U6-S0-Pad14) -> /4to1mux/QG_06
- U6 pad 2: unconnected-(U6-S1-Pad2) -> /4to1mux/QH_07
- U7 pad 14: unconnected-(U7-S0-Pad14) -> /4to1mux/QA_08
- U7 pad 2: unconnected-(U7-S1-Pad2) -> /4to1mux/QB_09
- U8 pad 14: unconnected-(U8-S0-Pad14) -> /4to1mux/QC_10
- U8 pad 2: unconnected-(U8-S1-Pad2) -> /4to1mux/QD_11

Commit message: Arduino: FPGA config bit working
Parts:
- removed U21: ESP32-WROOM-32E, RF_Module:ESP32-WROOM-32D
- added J2: Screw_Terminal_01x02, TerminalBlock:TerminalBlock_MaiXu_MX126-5.0-02P_1x02_P5.00mm, F.Cu at (135.8, 124.7)
- added U24: ~, buck_converter:Lm2596_buck, F.Cu at (139.2, 95.8)
- added U26: ATmega328-P, Package_DIP:DIP-28_W7.62mm, F.Cu at (210.9, 93.6)
- moved J1 87.4 mm to (98.8, 73.7)
- moved U19 81.2 mm to (118.0, 181.9)
- moved U1 81.2 mm to (58.9, 125.5)
- moved U10 81.2 mm to (9.93, 146.8)
- moved U17 81.2 mm to (94.8, 181.9)
- moved U2 81.2 mm to (74.6, 154.2)
- moved U20 81.2 mm to (129.5, 181.9)
- moved U24 81.2 mm to (184.6, 175.6)
- moved U5 81.2 mm to (78.1, 126.6)
- moved U6 81.2 mm to (-1.64, 122.9)
- moved U7 81.2 mm to (9.93, 122.9)
- moved U8 81.2 mm to (21.5, 122.9)
- moved U9 81.2 mm to (-1.64, 146.8)
- moved U11 81.2 mm to (-2.12, 188.5)
- moved U13 81.2 mm to (21.0, 188.5)
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Connections:
- U1 pad 12: Net-(U1-I7) -> /QH
- U1 pad 16: VCC -> Vout
- U10 pad 14: /SER -> /QH
- U10 pad 16: VCC -> Vout
- U10 pad 7: Net-(U10-QH) -> /QH1
- U11 pad 15: unconnected-(U11-Eb-Pad15) -> Vout
- U11 pad 16: VCC -> Vout
- U12 pad 15: unconnected-(U12-Eb-Pad15) -> Vout
- U12 pad 16: VCC -> Vout
- U13 pad 15: unconnected-(U13-Eb-Pad15) -> Vout
- U13 pad 16: VCC -> Vout
- U14 pad 15: unconnected-(U14-Eb-Pad15) -> Vout
- U14 pad 16: VCC -> Vout
- U15 pad 15: unconnected-(U15-Eb-Pad15) -> Vout
- U15 pad 16: VCC -> Vout
- U16 pad 15: unconnected-(U16-Eb-Pad15) -> Vout
- U16 pad 16: VCC -> Vout
- U17 pad 14: /SER -> /QH1
- U17 pad 16: VCC -> Vout
- U17 pad 7: Net-(U17-QH) -> /QH_2
- U18 pad 12: Net-(U17-QH) -> /QH_2
- U18 pad 16: VCC -> Vout
- U19 pad 14: /SER -> /QH_2
- U19 pad 16: VCC -> Vout
- U2 pad 15: unconnected-(U2-Eb-Pad15) -> Vout
- U2 pad 16: VCC -> Vout
- U20 pad 16: VCC -> Vout
- U22 pad 16: VCC -> Vout
- U23 pad 16: VCC -> Vout
- U25 pad 16: VCC -> Vout
- U3 pad 15: unconnected-(U3-Eb-Pad15) -> Vout
- U3 pad 16: VCC -> Vout
- U4 pad 15: unconnected-(U4-Eb-Pad15) -> Vout
- U4 pad 16: VCC -> Vout
- U5 pad 16: VCC -> Vout
- U5 pad 7: Net-(U1-I7) -> /QH
- U6 pad 15: unconnected-(U6-Eb-Pad15) -> Vout
- U6 pad 16: VCC -> Vout
- U7 pad 15: unconnected-(U7-Eb-Pad15) -> Vout
- U7 pad 16: VCC -> Vout
- U8 pad 15: unconnected-(U8-Eb-Pad15) -> Vout
- U8 pad 16: VCC -> Vout
- U9 pad 12: Net-(U10-QH) -> /QH1
- U9 pad 16: VCC -> Vout
Other:
- board outline added: 100 x 100 mm

Commit message: migrated stm32 compiler code to esp32 (no bitstream yet)
Parts:
- removed the U24 at (139.2, 95.8)
- removed U26: ATmega328-P, Package_DIP:DIP-28_W7.62mm
- added U21: DEVKIT_V1_ESP32-WROOM-32, ESP32_devkit:MODULE_DEVKIT_V1_ESP32-WROOM-32, F.Cu at (67.2, 40.3)
- J2: value Screw_Terminal_01x02 -> Conn_01x08_Pin; footprint TerminalBlock:TerminalBlock_MaiXu_MX126-5.0-02P_1x02_P5.00mm -> Connector_JST:JST_EH_B8B-EH-A_1x08_P2.50mm_Vertical
- moved U6 372.6 mm to (349.2, 248.3)
- moved U7 372.6 mm to (360.8, 248.3)
- moved U8 372.6 mm to (372.4, 248.3)
- moved U11 369.5 mm to (352.1, 293.9)
- moved U12 369.5 mm to (363.6, 293.9)
- moved U13 369.5 mm to (375.2, 293.9)
- moved U14 369.5 mm to (386.8, 293.9)
- moved U15 369.5 mm to (398.3, 293.9)
- moved U16 369.5 mm to (409.9, 293.9)
- moved U4 197.4 mm to (266.0, 276.8)
- moved U3 193.7 mm to (245.0, 276.3)
- moved U2 193.4 mm to (224.2, 276.8)
- moved J1 181.6 mm to (-27.2, 204.5)
- moved U10 170.0 mm to (163.3, 73.5)
- moved J2 142.6 mm to (16.2, 47.0), turned to 90 degrees
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Connections:
- J2 pad 1: /Gnd -> Vout
- J2 pad 2: /Vin -> GND
- U10 pad 10: unconnected-(U10-~{SRCLR}-Pad10) -> Vout
Routing:
- net Vout: track 0.00 -> 77.9 mm
- net /SER: track 0.00 -> 72.7 mm
- net /RCLK: track 0.00 -> 69.2 mm
- net /SRCLK: track 0.00 -> 64.7 mm
- net SER_sc: track 0.00 -> 52.0 mm
- net SRCLK_sc: track 0.00 -> 47.9 mm
- net RCLK_sc: track 0.00 -> 43.8 mm
- added copper zone on B.Cu, net GND
Other:
- board size 100 x 100 mm -> 248.9 x 97.9 mm

Commit message: PCB Designed for all the schematics
Parts:
- removed U24: 74HC595, Package_DIP:DIP-16_W7.62mm_LongPads
- added D1: LED, LED_THT:LED_D3.0mm, F.Cu at (863.5, 22.6)
- added D2: LED, LED_THT:LED_D3.0mm, F.Cu at (863.7, -29.7)
- added D3: LED, LED_THT:LED_D3.0mm, F.Cu at (863.5, -3.58)
- added D4: LED, LED_THT:LED_D3.0mm, F.Cu at (863.7, -52.5)
- added J10: Conn_01x03_Socket, Connector_PinSocket_2.54mm:PinSocket_1x03_P2.54mm_Vertical, F.Cu at (867.7, -68.9)
- added J11: Conn_01x05_Socket, Connector_PinHeader_2.54mm:PinHeader_1x05_P2.54mm_Vertical, F.Cu at (792.8, -106.3)
- added J12: Conn_01x05_Socket, Connector_PinHeader_2.54mm:PinHeader_1x05_P2.54mm_Vertical, F.Cu at (154.4, 152.7)
- added J3: Conn_01x08_Pin, Connector_PinSocket_2.54mm:PinSocket_1x08_P2.54mm_Vertical, F.Cu at (821.9, -22.4)
- added J4: Conn_01x08_Pin, Connector_PinSocket_2.54mm:PinSocket_1x08_P2.54mm_Vertical, F.Cu at (822.0, 23.9)
- added J5: Conn_01x08_Pin, Connector_PinSocket_2.54mm:PinSocket_1x08_P2.54mm_Vertical, F.Cu at (821.9, 1.06)
- added J6: Conn_01x08_Pin, Connector_PinSocket_2.54mm:PinSocket_1x08_P2.54mm_Vertical, F.Cu at (821.9, -45.5)
- added J7: Conn_01x03_Socket, Connector_PinSocket_2.54mm:PinSocket_1x03_P2.54mm_Vertical, F.Cu at (867.4, 2.47)
- added J8: Conn_01x03_Socket, Connector_PinSocket_2.54mm:PinSocket_1x03_P2.54mm_Vertical, F.Cu at (867.5, -19.9)
- added J9: Conn_01x03_Socket, Connector_PinSocket_2.54mm:PinSocket_1x03_P2.54mm_Vertical, F.Cu at (867.6, -44.1)
- J2: value Conn_01x08_Pin -> Conn_01x08_Socket; footprint Connector_JST:JST_EH_B8B-EH-A_1x08_P2.50mm_Vertical -> Connector_PinSocket_2.54mm:PinSocket_1x08_P2.54mm_Vertical
- U21: value DEVKIT_V1_ESP32-WROOM-32 -> ESP32-DEVKITC-32UE; footprint ESP32_devkit:MODULE_DEVKIT_V1_ESP32-WROOM-32 -> ESP32_devkit:ESPRESSIF_ESP32-DEVKITC-32UE
- moved U9 895.5 mm to (835.3, -3.43), turned to 90 degrees
- moved U1 833.8 mm to (835.4, 18.9), turned to 90 degrees
- moved U18 804.7 mm to (835.3, -28.2), turned to 90 degrees
- moved U20 788.3 mm to (835.4, -51.2), turned to 90 degrees
- moved U21 779.3 mm to (845.3, 83.6), turned to 90 degrees
- moved J2 778.5 mm to (793.5, 90.5), turned to 180 degrees
- moved U5 651.6 mm to (789.5, 13.9), turned to 90 degrees
- moved U10 632.4 mm to (789.6, -14.4), turned to 90 degrees
- moved U17 617.1 mm to (789.7, -45.8), turned to 90 degrees
- moved U19 605.0 mm to (789.9, -79.7), turned to 90 degrees
- moved U11 366.2 mm to (42.1, 98.8)
- moved U12 357.7 mm to (63.5, 99.2)
- moved U13 350.2 mm to (84.0, 99.2)
- moved U14 341.1 mm to (106.7, 99.2)
- moved U15 332.3 mm to (128.9, 99.3)
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Connections:
- U10 pad 13: /OE_1 -> GND
- U17 pad 10: unconnected-(U17-~{SRCLR}-Pad10) -> Vout
- U17 pad 13: /OE_2 -> GND
- U19 pad 10: unconnected-(U19-~{SRCLR}-Pad10) -> Vout
- U19 pad 13: /OE_3 -> GND
- U21 pad 10: SRCLK_sc -> unconnected-(U21-26-Pad10)
- U21 pad 11: RCLK_sc -> unconnected-(U21-27-Pad11)
- U21 pad 12: unconnected-(U21-RX0-Pad12) -> SER_sc
- U21 pad 13: unconnected-(U21-TX0-Pad13) -> /SRCLK
- U21 pad 14: unconnected-(U21-D22-Pad14) -> GND
- U21 pad 15: unconnected-(U21-D23-Pad15) -> /RCLK
- U21 pad 19: unconnected-(U21-D34-Pad19) -> Vout
- U21 pad 2: GND -> unconnected-(U21-EN-Pad2)
- U21 pad 20: unconnected-(U21-D35-Pad20) -> GND
- U21 pad 26: /SRCLK -> GND
- U21 pad 28: /SER -> unconnected-(U21-18-Pad28)
- U21 pad 29: GND -> /SER
- U21 pad 3: /RCLK -> unconnected-(U21-VP-Pad3)
- U21 pad 30: Vout -> unconnected-(U21-17-Pad30)
- U21 pad 9: SER_sc -> unconnected-(U21-25-Pad9)
- U5 pad 10: unconnected-(U5-~{SRCLR}-Pad10) -> Vout
- U5 pad 13: /OE_0 -> GND
Routing:
- net GND: track 0.00 -> 492.2 mm, vias 0 -> 49
- net Vout: track 77.9 -> 466.5 mm, vias 0 -> 31
- net /4to1mux/QH_07: track 0.00 -> 146.8 mm, vias 0 -> 2
- net /4to1mux/QB_01: track 0.00 -> 122.4 mm
- net /4to1mux/QG_06: track 0.00 -> 108.3 mm, vias 0 -> 2
- net /4to1mux/QD_11: track 0.00 -> 107.9 mm, vias 0 -> 2
- net /4to1mux/QC_10: track 0.00 -> 102.8 mm, vias 0 -> 2
- net Net-(J6-Pin_1): track 0.00 -> 97.1 mm
- net SER_sc: track 52.0 -> 148.8 mm, vias 0 -> 2
- net Net-(J3-Pin_1): track 0.00 -> 89.4 mm
- net /4to1mux/QF_05: track 0.00 -> 89.4 mm, vias 0 -> 2
- net Net-(J4-Pin_1): track 0.00 -> 87.6 mm
- net /4to1mux/QA_00: track 0.00 -> 85.3 mm
- net /4to1mux/QE_04: track 0.00 -> 84.3 mm, vias 0 -> 2
- net Net-(J5-Pin_1): track 0.00 -> 84.0 mm
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- added copper zone on B.Cu, net Vout
Other:
- board size 248.9 x 97.9 mm -> 850.2 x 267.4 mm
